Commit message: last

File: source/FABRICS/src/fabrics_sim/models/robots/urdf/openarm_tesollo/openarm_tesollo.urdf (robot description, URDF)
Before this commit: robot open_tesollo, 57 links, 56 joints
Joints:
- joint rj_dg_1_1: origin xyz=-0.0162 0.019 0.0866 rpy=0. 0. 0. -> xyz=-0.0162 0.019 0.0128 rpy=0. 0. 0.
- joint rj_dg_2_1: origin xyz=-0.0071 0.027 0.1399 rpy=0. 0. 0. -> xyz=-0.0071 0.027 0.0661 rpy=0. 0. 0.
- joint rj_dg_3_1: origin xyz=-0.0071 0.0025 0.1439 rpy=0. 0. 0. -> xyz=-0.0071 0.0025 0.0701 rpy=0. 0. 0.
- joint rj_dg_4_1: origin xyz=-0.0071 -0.022 0.1359 rpy=0. 0. 0. -> xyz=-0.0071 -0.022 0.0621 rpy=0. 0. 0.
- joint rj_dg_5_1: origin xyz=0.0103 -0.0195 0.092  rpy=0. 0. 0. -> xyz=0.0103 -0.0195 0.0182 rpy=0. 0. 0.
