Commit message: feat(fabrics): dg5f-m 양팔 fabric 자산 + 손가락 반발쌍
09.05 자산 라인업(openarm_dg5f-m_bi_rl)에 맞는 fabric URDF·params 를 추가한다.
구 `openarm_tesollo_sensor_right` 와 **완전 드롭인**이다 — 링크 이름 104개, 구동관절
27개 순서, body_repulsion 충돌구 프레임 65개가 전부 일치한다(이관 전 대조 확인).

- `models/robots/urdf/openarm_dg5f-m_bi_{left,right}` + 공유 메시 심볼릭 링크
- `fabric_params/openarm_dg5f-m_{left,right}_pose_params.yaml`
  구 params 대비 `collision_link_prefix_pairs` 가 16 → 176 으로 늘었다(손가락끼리
  160쌍 추가). 팔 그룹의 자기충돌은 여전히 비활성이므로 실제 발동은 손 그룹
  (`use_hand_repulsion`)을 켤 때다.
- `openarm_tesollo_pose_fabric.py`: 반발 그룹을 팔·손으로 나누는 구성 정리
- `assets/simulation_setting/shaker`: sim 메시와 같은 물체의 FP++ CAD

Co-Authored-By: Claude Opus 5 <noreply@anthropic.com>
Claude-Session: https://claude.ai/code/session_01X3UjBxvcdQMDLsryR8e6J6

File: source/FABRICS/src/fabrics_sim/models/robots/urdf/openarm_dg5f-m_bi_left/openarm_dg5f-m_bi_left.urdf (robot description, URDF)
Before this commit: robot openarm_dg5f-m_bi_left, 62 links, 61 joints
Links:
- removed link tesollo_right_rl_dg_1_1_sphere2
- removed link tesollo_right_rl_dg_1_3_sphere2
- removed link tesollo_right_rl_dg_2_1_sphere2
- removed link tesollo_right_rl_dg_2_3_sphere2
- removed link tesollo_right_rl_dg_3_1_sphere2
- removed link tesollo_right_rl_dg_3_3_sphere2
- removed link tesollo_right_rl_dg_4_1_sphere2
- removed link tesollo_right_rl_dg_4_3_sphere2
- removed link tesollo_right_rl_dg_5_1_sphere2
- removed link tesollo_right_rl_dg_5_3_sphere2
- added link tesollo_right_rl_dg_1_1_sph1, mass 0.001
- added link tesollo_right_rl_dg_1_1_sph2, mass 0.001
- added link tesollo_right_rl_dg_1_1_sph3, mass 0.001
- added link tesollo_right_rl_dg_1_2_sph1, mass 0.001
- added link tesollo_right_rl_dg_1_2_sph2, mass 0.001
- added link tesollo_right_rl_dg_1_3_sph1, mass 0.001
- added link tesollo_right_rl_dg_1_3_sph2, mass 0.001
- added link tesollo_right_rl_dg_1_3_sph3, mass 0.001
- added link tesollo_right_rl_dg_1_4_sph1, mass 0.001
- added link tesollo_right_rl_dg_1_4_sph2, mass 0.001
- added link tesollo_right_rl_dg_1_4_sph3, mass 0.001
- added link tesollo_right_rl_dg_2_1_sph1, mass 0.001
- added link tesollo_right_rl_dg_2_1_sph2, mass 0.001
- added link tesollo_right_rl_dg_2_2_sph1, mass 0.001
- added link tesollo_right_rl_dg_2_2_sph2, mass 0.001
- added link tesollo_right_rl_dg_2_2_sph3, mass 0.001
- added link tesollo_right_rl_dg_2_3_sph1, mass 0.001
- added link tesollo_right_rl_dg_2_3_sph2, mass 0.001
- added link tesollo_right_rl_dg_2_3_sph3, mass 0.001
- added link tesollo_right_rl_dg_2_4_sph1, mass 0.001
- added link tesollo_right_rl_dg_2_4_sph2, mass 0.001
- added link tesollo_right_rl_dg_3_1_sph1, mass 0.001
- added link tesollo_right_rl_dg_3_1_sph2, mass 0.001
- added link tesollo_right_rl_dg_3_2_sph1, mass 0.001
- added link tesollo_right_rl_dg_3_2_sph2, mass 0.001
- added link tesollo_right_rl_dg_3_2_sph3, mass 0.001
- added link tesollo_right_rl_dg_3_3_sph1, mass 0.001
- added link tesollo_right_rl_dg_3_3_sph2, mass 0.001
- added link tesollo_right_rl_dg_3_3_sph3, mass 0.001
- added link tesollo_right_rl_dg_3_4_sph1, mass 0.001
- added link tesollo_right_rl_dg_3_4_sph2, mass 0.001
- added link tesollo_right_rl_dg_4_1_sph1, mass 0.001
- added link tesollo_right_rl_dg_4_1_sph2, mass 0.001
- added link tesollo_right_rl_dg_4_2_sph1, mass 0.001
- added link tesollo_right_rl_dg_4_2_sph2, mass 0.001
- added link tesollo_right_rl_dg_4_2_sph3, mass 0.001
- added link tesollo_right_rl_dg_4_3_sph1, mass 0.001
- added link tesollo_right_rl_dg_4_3_sph2, mass 0.001
- added link tesollo_right_rl_dg_4_3_sph3, mass 0.001
- added link tesollo_right_rl_dg_4_4_sph1, mass 0.001
- added link tesollo_right_rl_dg_4_4_sph2, mass 0.001
- added link tesollo_right_rl_dg_5_1_sph1, mass 0.001
- added link tesollo_right_rl_dg_5_1_sph2, mass 0.001
- added link tesollo_right_rl_dg_5_1_sph3, mass 0.001
- added link tesollo_right_rl_dg_5_2_sph1, mass 0.001
- added link tesollo_right_rl_dg_5_2_sph2, mass 0.001
- added link tesollo_right_rl_dg_5_3_sph1, mass 0.001
- added link tesollo_right_rl_dg_5_3_sph2, mass 0.001
- added link tesollo_right_rl_dg_5_3_sph3, mass 0.001
- added link tesollo_right_rl_dg_5_4_sph1, mass 0.001
- added link tesollo_right_rl_dg_5_4_sph2, mass 0.001
- added link tesollo_right_rl_dg_5_4_sph3, mass 0.001
Joints:
- removed joint tesollo_right_rl_dg_1_1_joint_sphere2
- removed joint tesollo_right_rl_dg_1_3_joint_sphere2
- removed joint tesollo_right_rl_dg_2_1_joint_sphere2
- removed joint tesollo_right_rl_dg_2_3_joint_sphere2
- removed joint tesollo_right_rl_dg_3_1_joint_sphere2
- removed joint tesollo_right_rl_dg_3_3_joint_sphere2
- removed joint tesollo_right_rl_dg_4_1_joint_sphere2
- removed joint tesollo_right_rl_dg_4_3_joint_sphere2
- removed joint tesollo_right_rl_dg_5_1_joint_sphere2
- removed joint tesollo_right_rl_dg_5_3_joint_sphere2
- added joint tesollo_right_rl_dg_1_1_sph1_joint: type fixed, parent tesollo_right_rl_dg_1_1, child tesollo_right_rl_dg_1_1_sph1, origin xyz=0.006992 0.000000 0.000000 rpy=0. 0. 0.
- added joint tesollo_right_rl_dg_1_1_sph2_joint: type fixed, parent tesollo_right_rl_dg_1_1, child tesollo_right_rl_dg_1_1_sph2, origin xyz=0.020975 0.000000 0.000000 rpy=0. 0. 0.
- added joint tesollo_right_rl_dg_1_1_sph3_joint: type fixed, parent tesollo_right_rl_dg_1_1, child tesollo_right_rl_dg_1_1_sph3, origin xyz=0.034958 0.000000 0.000000 rpy=0. 0. 0.
- added joint tesollo_right_rl_dg_1_2_sph1_joint: type fixed, parent tesollo_right_rl_dg_1_2, child tesollo_right_rl_dg_1_2_sph1, origin xyz=0.000000 -0.007750 0.000000 rpy=0. 0. 0.
- added joint tesollo_right_rl_dg_1_2_sph2_joint: type fixed, parent tesollo_right_rl_dg_1_2, child tesollo_right_rl_dg_1_2_sph2, origin xyz=0.000000 -0.023250 0.000000 rpy=0. 0. 0.
- added joint tesollo_right_rl_dg_1_3_sph1_joint: type fixed, parent tesollo_right_rl_dg_1_3, child tesollo_right_rl_dg_1_3_sph1, origin xyz=0.000000 -0.006467 0.000000 rpy=0. 0. 0.
- added joint tesollo_right_rl_dg_1_3_sph2_joint: type fixed, parent tesollo_right_rl_dg_1_3, child tesollo_right_rl_dg_1_3_sph2, origin xyz=0.000000 -0.019400 0.000000 rpy=0. 0. 0.
- added joint tesollo_right_rl_dg_1_3_sph3_joint: type fixed, parent tesollo_right_rl_dg_1_3, child tesollo_right_rl_dg_1_3_sph3, origin xyz=0.000000 -0.032333 0.000000 rpy=0. 0. 0.
- added joint tesollo_right_rl_dg_1_4_sph1_joint: type fixed, parent tesollo_right_rl_dg_1_4, child tesollo_right_rl_dg_1_4_sph1, origin xyz=0.000000 -0.006050 0.000000 rpy=0. 0. 0.
- added joint tesollo_right_rl_dg_1_4_sph2_joint: type fixed, parent tesollo_right_rl_dg_1_4, child tesollo_right_rl_dg_1_4_sph2, origin xyz=0.000000 -0.018150 0.000000 rpy=0. 0. 0.
- added joint tesollo_right_rl_dg_1_4_sph3_joint: type fixed, parent tesollo_right_rl_dg_1_4, child tesollo_right_rl_dg_1_4_sph3, origin xyz=0.000000 -0.030250 0.000000 rpy=0. 0. 0.
- added joint tesollo_right_rl_dg_2_1_sph1_joint: type fixed, parent tesollo_right_rl_dg_2_1, child tesollo_right_rl_dg_2_1_sph1, origin xyz=0.004412 0.000000 0.006625 rpy=0. 0. 0.
- added joint tesollo_right_rl_dg_2_1_sph2_joint: type fixed, parent tesollo_right_rl_dg_2_1, child tesollo_right_rl_dg_2_1_sph2, origin xyz=0.013237 0.000000 0.019875 rpy=0. 0. 0.
- added joint tesollo_right_rl_dg_2_2_sph1_joint: type fixed, parent tesollo_right_rl_dg_2_2, child tesollo_right_rl_dg_2_2_sph1, origin xyz=0.000000 0.000000 0.006467 rpy=0. 0. 0.
- added joint tesollo_right_rl_dg_2_2_sph2_joint: type fixed, parent tesollo_right_rl_dg_2_2, child tesollo_right_rl_dg_2_2_sph2, origin xyz=0.000000 0.000000 0.019400 rpy=0. 0. 0.
- added joint tesollo_right_rl_dg_2_2_sph3_joint: type fixed, parent tesollo_right_rl_dg_2_2, child tesollo_right_rl_dg_2_2_sph3, origin xyz=0.000000 0.000000 0.032333 rpy=0. 0. 0.
- added joint tesollo_right_rl_dg_2_3_sph1_joint: type fixed, parent tesollo_right_rl_dg_2_3, child tesollo_right_rl_dg_2_3_sph1, origin xyz=0.000000 0.000000 0.006467 rpy=0. 0. 0.
- added joint tesollo_right_rl_dg_2_3_sph2_joint: type fixed, parent tesollo_right_rl_dg_2_3, child tesollo_right_rl_dg_2_3_sph2, origin xyz=0.000000 0.000000 0.019400 rpy=0. 0. 0.
- added joint tesollo_right_rl_dg_2_3_sph3_joint: type fixed, parent tesollo_right_rl_dg_2_3, child tesollo_right_rl_dg_2_3_sph3, origin xyz=0.000000 0.000000 0.032333 rpy=0. 0. 0.
- added joint tesollo_right_rl_dg_2_4_sph1_joint: type fixed, parent tesollo_right_rl_dg_2_4, child tesollo_right_rl_dg_2_4_sph1, origin xyz=0.000000 0.000000 0.006375 rpy=0. 0. 0.
- added joint tesollo_right_rl_dg_2_4_sph2_joint: type fixed, parent tesollo_right_rl_dg_2_4, child tesollo_right_rl_dg_2_4_sph2, origin xyz=0.000000 0.000000 0.019125 rpy=0. 0. 0.
- added joint tesollo_right_rl_dg_3_1_sph1_joint: type fixed, parent tesollo_right_rl_dg_3_1, child tesollo_right_rl_dg_3_1_sph1, origin xyz=0.004412 0.000000 0.006625 rpy=0. 0. 0.
- added joint tesollo_right_rl_dg_3_1_sph2_joint: type fixed, parent tesollo_right_rl_dg_3_1, child tesollo_right_rl_dg_3_1_sph2, origin xyz=0.013237 0.000000 0.019875 rpy=0. 0. 0.
- added joint tesollo_right_rl_dg_3_2_sph1_joint: type fixed, parent tesollo_right_rl_dg_3_2, child tesollo_right_rl_dg_3_2_sph1, origin xyz=0.000000 0.000000 0.006467 rpy=0. 0. 0.
- added joint tesollo_right_rl_dg_3_2_sph2_joint: type fixed, parent tesollo_right_rl_dg_3_2, child tesollo_right_rl_dg_3_2_sph2, origin xyz=0.000000 0.000000 0.019400 rpy=0. 0. 0.
- added joint tesollo_right_rl_dg_3_2_sph3_joint: type fixed, parent tesollo_right_rl_dg_3_2, child tesollo_right_rl_dg_3_2_sph3, origin xyz=0.000000 0.000000 0.032333 rpy=0. 0. 0.
- added joint tesollo_right_rl_dg_3_3_sph1_joint: type fixed, parent tesollo_right_rl_dg_3_3, child tesollo_right_rl_dg_3_3_sph1, origin xyz=0.000000 0.000000 0.006467 rpy=0. 0. 0.
- added joint tesollo_right_rl_dg_3_3_sph2_joint: type fixed, parent tesollo_right_rl_dg_3_3, child tesollo_right_rl_dg_3_3_sph2, origin xyz=0.000000 0.000000 0.019400 rpy=0. 0. 0.
- added joint tesollo_right_rl_dg_3_3_sph3_joint: type fixed, parent tesollo_right_rl_dg_3_3, child tesollo_right_rl_dg_3_3_sph3, origin xyz=0.000000 0.000000 0.032333 rpy=0. 0. 0.
- added joint tesollo_right_rl_dg_3_4_sph1_joint: type fixed, parent tesollo_right_rl_dg_3_4, child tesollo_right_rl_dg_3_4_sph1, origin xyz=0.000000 0.000000 0.006375 rpy=0. 0. 0.
- added joint tesollo_right_rl_dg_3_4_sph2_joint: type fixed, parent tesollo_right_rl_dg_3_4, child tesollo_right_rl_dg_3_4_sph2, origin xyz=0.000000 0.000000 0.019125 rpy=0. 0. 0.
- added joint tesollo_right_rl_dg_4_1_sph1_joint: type fixed, parent tesollo_right_rl_dg_4_1, child tesollo_right_rl_dg_4_1_sph1, origin xyz=0.004412 0.000000 0.006625 rpy=0. 0. 0.
- added joint tesollo_right_rl_dg_4_1_sph2_joint: type fixed, parent tesollo_right_rl_dg_4_1, child tesollo_right_rl_dg_4_1_sph2, origin xyz=0.013237 0.000000 0.019875 rpy=0. 0. 0.
- added joint tesollo_right_rl_dg_4_2_sph1_joint: type fixed, parent tesollo_right_rl_dg_4_2, child tesollo_right_rl_dg_4_2_sph1, origin xyz=0.000000 0.000000 0.006467 rpy=0. 0. 0.
- added joint tesollo_right_rl_dg_4_2_sph2_joint: type fixed, parent tesollo_right_rl_dg_4_2, child tesollo_right_rl_dg_4_2_sph2, origin xyz=0.000000 0.000000 0.019400 rpy=0. 0. 0.
- added joint tesollo_right_rl_dg_4_2_sph3_joint: type fixed, parent tesollo_right_rl_dg_4_2, child tesollo_right_rl_dg_4_2_sph3, origin xyz=0.000000 0.000000 0.032333 rpy=0. 0. 0.
- added joint tesollo_right_rl_dg_4_3_sph1_joint: type fixed, parent tesollo_right_rl_dg_4_3, child tesollo_right_rl_dg_4_3_sph1, origin xyz=0.000000 0.000000 0.006467 rpy=0. 0. 0.
- added joint tesollo_right_rl_dg_4_3_sph2_joint: type fixed, parent tesollo_right_rl_dg_4_3, child tesollo_right_rl_dg_4_3_sph2, origin xyz=0.000000 0.000000 0.019400 rpy=0. 0. 0.
- added joint tesollo_right_rl_dg_4_3_sph3_joint: type fixed, parent tesollo_right_rl_dg_4_3, child tesollo_right_rl_dg_4_3_sph3, origin xyz=0.000000 0.000000 0.032333 rpy=0. 0. 0.
- added joint tesollo_right_rl_dg_4_4_sph1_joint: type fixed, parent tesollo_right_rl_dg_4_4, child tesollo_right_rl_dg_4_4_sph1, origin xyz=0.000000 0.000000 0.006375 rpy=0. 0. 0.
- added joint tesollo_right_rl_dg_4_4_sph2_joint: type fixed, parent tesollo_right_rl_dg_4_4, child tesollo_right_rl_dg_4_4_sph2, origin xyz=0.000000 0.000000 0.019125 rpy=0. 0. 0.
- added joint tesollo_right_rl_dg_5_1_sph1_joint: type fixed, parent tesollo_right_rl_dg_5_1, child tesollo_right_rl_dg_5_1_sph1, origin xyz=0.000000 0.004667 0.006350 rpy=0. 0. 0.
- added joint tesollo_right_rl_dg_5_1_sph2_joint: type fixed, parent tesollo_right_rl_dg_5_1, child tesollo_right_rl_dg_5_1_sph2, origin xyz=0.000000 0.014000 0.019050 rpy=0. 0. 0.
- added joint tesollo_right_rl_dg_5_1_sph3_joint: type fixed, parent tesollo_right_rl_dg_5_1, child tesollo_right_rl_dg_5_1_sph3, origin xyz=0.000000 0.023333 0.031750 rpy=0. 0. 0.
- added joint tesollo_right_rl_dg_5_2_sph1_joint: type fixed, parent tesollo_right_rl_dg_5_2, child tesollo_right_rl_dg_5_2_sph1, origin xyz=0.000000 0.000000 0.007750 rpy=0. 0. 0.
- added joint tesollo_right_rl_dg_5_2_sph2_joint: type fixed, parent tesollo_right_rl_dg_5_2, child tesollo_right_rl_dg_5_2_sph2, origin xyz=0.000000 0.000000 0.023250 rpy=0. 0. 0.
- added joint tesollo_right_rl_dg_5_3_sph1_joint: type fixed, parent tesollo_right_rl_dg_5_3, child tesollo_right_rl_dg_5_3_sph1, origin xyz=0.000000 0.000000 0.006467 rpy=0. 0. 0.
- added joint tesollo_right_rl_dg_5_3_sph2_joint: type fixed, parent tesollo_right_rl_dg_5_3, child tesollo_right_rl_dg_5_3_sph2, origin xyz=0.000000 0.000000 0.019400 rpy=0. 0. 0.
- added joint tesollo_right_rl_dg_5_3_sph3_joint: type fixed, parent tesollo_right_rl_dg_5_3, child tesollo_right_rl_dg_5_3_sph3, origin xyz=0.000000 0.000000 0.032333 rpy=0. 0. 0.
- added joint tesollo_right_rl_dg_5_4_sph1_joint: type fixed, parent tesollo_right_rl_dg_5_4, child tesollo_right_rl_dg_5_4_sph1, origin xyz=0.000000 0.000000 0.006050 rpy=0. 0. 0.
- added joint tesollo_right_rl_dg_5_4_sph2_joint: type fixed, parent tesollo_right_rl_dg_5_4, child tesollo_right_rl_dg_5_4_sph2, origin xyz=0.000000 0.000000 0.018150 rpy=0. 0. 0.
- added joint tesollo_right_rl_dg_5_4_sph3_joint: type fixed, parent tesollo_right_rl_dg_5_4, child tesollo_right_rl_dg_5_4_sph3, origin xyz=0.000000 0.000000 0.030250 rpy=0. 0. 0.
